File: project_files/Ohmsprint.kicad_sch (KiCad schematic)
At the start: 74 parts, among them J1 USB_C_Receptacle_USB2.0_16P, J3 PJ-002AH-SMT-TR, J4 SJ-3523-SMT-TR, Q1 SS8050, Q2 SS8050, SW1 SW_Push, SW2 SW_Push, U1 CP2102N-Axx-xQFN28, U2 ESP32-WROOM-32, U3 AMS1117-3.3, U4 ATM90E26-YU, U5 ABS210-13, Y1 8.192MHz

Commit message: Buck konvertor, jumperi, SPI, DigiKey proizvodi
Parts:
- removed C1: 4u7/6V3 10%, symbol Device:C
- removed C11: 47u/16V Tant, symbol Device:C
- removed C2: 100n/50V 10%, symbol Device:C
- removed C25: 22u/10V Tant, symbol Device:C
- removed C3: 1uF/16V(10%), symbol Device:C
- removed C6: 100n/50V 10%, symbol Device:C_Small
- removed C9: 10u, symbol Device:C_Small
- removed R13: 10k 5%, symbol Device:R_US
- removed R25, R26: 1k, symbol Device:R_US
- removed U1: CP2102N-Axx-xQFN28, Package_DFN_QFN:QFN-28-1EP_5x5mm_P0.5mm_EP3.35x3.35mm, symbol Interface_USB:CP2102N-Axx-xQFN28
- removed U2: ESP32-WROOM-32, RF_Module:ESP32-WROOM-32, symbol RF_Module:ESP32-WROOM-32
- removed U3: AMS1117-3.3, Package_TO_SOT_SMD:SOT-223-3_TabPin2, symbol Regulator_Linear:AMS1117-3.3
- added C1: 1u, symbol Device:C_Small
- added C10: 4u7/6V3, symbol Device:C
- added C11: 47u Elec, symbol Device:C_Polarized
- added C2: 47u Tant, symbol Device:C_Polarized
- added C20: 0.1u/50V, symbol Device:C
- added C25: 100p, symbol Device:C_Small
- added C27: 1uF/16V(10%), symbol Device:C
- added C28, C29, C9: 22u, symbol Device:C_Polarized
- added C3: 10u Al Elec, symbol Device:C_Polarized
- added C30: 100n, symbol Device:C_Small
- added C6: 10u Tant, symbol Device:C_Polarized
- added JP6, JP7: Default Connected, symbol Jumper:SolderJumper_2_Open
- added JP8, JP9: 2+3, symbol Jumper:SolderJumper_3_Open
- added L1: 10u, symbol Device:L
- added R31: 22k1 1%, symbol Device:R_US
- added R32: 47k5 1%, symbol Device:R_US
- added R33: 2k (5%), symbol Device:R_US
- added U1: ESP32-WROOM-32E, RF_Module:ESP32-WROOM-32D, symbol RF_Module:ESP32-WROOM-32E
- added U2: AP63203WU, Package_TO_SOT_SMD:TSOT-23-6, symbol Regulator_Switching:AP63203WU
- added U3: MIC29302AWD, Package_TO_SOT_SMD:TO-252-5_TabPin3, symbol Regulator_Linear:MIC29302AWD
- added U6: CP2102N-A02-GQFN28, QFN28_5X5_SIL, symbol cp2102n-a02-gqfn28:CP2102N-A02-GQFN28
- C16: value 10n -> 1n
- C4: value 100n/50V 10% NC -> 0.1u DNP
- C5: value 100n/50V 10% -> 0.1u DNP
- C7: value 22u/10V 20% -> 100n
- R10: value 0 -> 200k
- R14, R15: value 10k 5% -> 10k
- R16, R27: value 3k -> 4k2
- R17, R18: value 4k2 -> 3k
- R6: value 22k1 1% -> 0
- R7: value 47k5 1% -> 100
- R8: value 2k (5%) -> 166
- R9: value 0 -> 50k
Connections:
- net I2N is gone; now on net GND: U4.8 (I2N)
- net I2P is gone; now on net GND: U4.7 (I2P)
- net +3.3V: now also C26.1, R6.2, R7.1, C10.1, C11.1, C20.1, C3.1, C9.1, JP8.1 (A), JP9.3 (B), R33.1, U1.2 (VDD), U3.4 (VOUT), U6.6 (VDD), U6.7 (VREGIN); no longer C13.1, C7.1, R8.1, U4.28 (MMD0), U4.5 (AVDD)
- net CS: now also U1.29 (IO5)
- net DTR: now also U6.28 (DTR)
- net Data+: now also U6.4 (D+)
- net Data-: now also U6.5 (D-)
- net EN: now also C1.1, U1.3 (EN)
- net GND: now also R10.2, R8.2, C1.2, C10.2, C11.2, C2.2, C20.2, C27.2, C28.2, C29.2, C3.2, C30.2, C6.2, C9.2, JP8.3 (B), JP9.1 (A), R32.2, U1.1 (GND), U1.15 (GND), U1.38 (GND), U1.39 (GND), U2.4 (GND), U3.3 (GND), U6.29 (GND), U6.3 (GND); no longer C7.2, R7.2, U4.1 (MMD1)
- net IO0: now also U1.25 (IO0)
- net MISO: now also U1.31 (IO19)
- net MOSI: now also U1.37 (IO23)
- net RTS: now also U6.24 (RTS)
- net RXD0: now also JP7.2 (B), U1.34 (RXD0/IO3); no longer R10.2
- net SCLK: now also U1.30 (IO18)
- net TXD0: now also JP6.2 (B), U1.35 (TXD0/IO1); no longer R9.2
- net VBUS: now also C27.1, R31.1; no longer R6.1
- net WarnOut: now also U1.14 (IO12)
- net ~4V Merni: now reaches R9.1
- net ~4V Merni: now also JP3.1 (A), C25.1, C28.1, C29.1, L1.2
- net at R10.1: now also R9.2, C25.2, U2.1 (FB)
- net ATIM_CF1: now reaches U4.18 (CF1)
- net ATIM_CF1: now also U1.9 (IO33)
- net ATM_CF2: now reaches U4.19 (CF2)
- net ATM_CF2: now also U1.8 (IO32)
- net ATM_IRQ: now reaches U4.20 (IRQ)
- net ATM_IRQ: now also U1.13 (IO14)
- net ATM_ZX: now reaches U4.21 (ZX)
- net ATM_ZX: now also U1.12 (IO27)
- net +5V: no longer names the net of C24.1, JP3.2 (C), R1.1
- net +5V: now also C2.1, U3.1 (EN), U3.2 (VIN)
- net 7V Merni: no longer names the net of U5.1
- net 7V Merni: now also C30.1, C6.1, U2.2 (EN), U2.3 (IN); no longer JP3.1 (A)
- new net: R7.2, R8.1, U3.5 (ADJ)
- new net: C13.1, R6.1, U4.5 (AVDD)
- new net: R33.2, U6.9 (RSTb)
- new net: C7.1, U2.6 (BST)
- new net: C7.2, L1.1, U2.5 (SW)
- new net: JP8.2 (C), U4.1 (MMD1)
- new net: JP7.1 (A), U6.26 (TXD)
- new net: JP9.2 (C), U4.28 (MMD0)
- new net: JP6.1 (A), U6.25 (RXD)
- new net VBUS-3.3: R31.2, R32.1, U6.8 (VBUS)
Other:
- note added: "Alternativa AMS1117-3.3"
- note added: "Alternativa CH340"
- note added: "Alternativne opcije za buck su AP63205WU, koji daje 5V na izlazu, LM2596-5, koji isto daje 5V na izlazu."
- note added: "Bilo bi dobro da se nadje verzija sa fiksnim izlaznim naponom a da nije preko 5 evra"
- note added: "Kondenzatori od 0.1u, 1u, 10u"
- note added: "Moramo imati buck konvertor jer je jedini nacin da vucemo preko 1A, a da ne zapalimo LDO. Cilj je da 4V iz buck-a dovedemo na LDO koji ce izbaciti stabilnih 3.3V bez switching noise koji bi smetao mernom chipu"
- note added: "Mozda nam ni ne treba LDO, moramo se dogovoriti, i dalje nisam siguran da li buck ima dovoljno mali noise"
- note added: "Pametno je groundovati ova dva pina jer mogu da pokupe i najmanji sum"
- note added: "Par otpornika od 33R, 10k"
- note added: "Pinovi za SPI su VSPI konfiguracija iz ESP dokumentacije"
- note added: "Proveriti datasheet za kombinacije"
- note added: "Viskovi"
- note removed: "?"
- note removed: "Ovi otpornici su tu kako bi mogli da se odleme za tesiranje. (Tako u svim semama stoji)"
- note removed: "Ovo je samo kako ne bi visili pinovi"
- note removed: "Uzmimo heatsink za regulator za svaki slucaj"
- moved on the sheet: C18, C19, C21, C22, C23, C24, C26, C4, C5, D1, D2, D3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

Commit message: Novi power supply, doradjena sema
Parts:
- removed C2: 47u Tant, symbol Device:C_Polarized
- removed C24, C26: 100n Ceram, symbol Device:C
- removed C25: 100p, symbol Device:C_Small
- removed JP3: Jumper_3_Open, symbol Jumper:Jumper_3_Open
- removed JP6, JP7: Default Connected, symbol Jumper:SolderJumper_2_Open
- removed R10: 200k, symbol Device:R_US
- removed R8: 166, symbol Device:R_US
- removed R9: 50k, symbol Device:R_US
- removed U3: MIC29302AWD, Package_TO_SOT_SMD:TO-252-5_TabPin3, symbol Regulator_Linear:MIC29302AWD
- added C24, C25: 10u Low ESR, symbol Device:C_Polarized
- added C26: 100n, symbol Device:C_Small
- added C31, C32: 22u, symbol Device:C_Polarized
- added D6: SMAJ12A, Diode_SMD:D_SMA, symbol Diode:SMAJ12A
- added D7: LED_RED, symbol Device:LED
- added JP1: Jumper_3_Open, symbol Jumper:Jumper_3_Open
- added L2: 4.7u, symbol Device:L
- added R10, R13, R25, R9: 33R, symbol Device:R_Small_US
- added R26, R28: 0R, symbol Device:R_Small_US
- added U3: AP63205WU, Package_TO_SOT_SMD:TSOT-23-6, symbol Regulator_Switching:AP63205WU
- added U7: MCP1727-3302xSN, Package_SO:SOIC-8_3.9x4.9mm_P1.27mm, symbol Regulator_Linear:MCP1727-3302xSN
- C3: value 10u Al Elec -> 22u Tant
- C6: value 10u Tant -> 470u Low ESR Electr
- D1: value LED_RED -> LED_GREEN
- L1: value 10u -> 3.9u
- R7: value 100 -> 2k
Connections:
- net ~4V Merni is gone; now on net +3.3VD: C28.1, C29.1, L1.2
- net GND: now also C24.2, C25.2, C31.2, C32.2, D6.2 (A2), D7.1 (K), U3.4 (GND), U7.4 (GND), U7.6 (Cdelay)
- net RXD0: now also R26.2
- net TXD0: now also R28.2
- net +3.3VA: now reaches R1.1
- net +3.3VA: now also C11.1, C12.1, C3.1, JP8.1 (A), JP9.3 (B), R6.2, U4.3 (DVDD), U7.7 (Sense), U7.8 (Vout)
- net at R7.2: now also D7.2 (A)
- net +3.3VD: now reaches U2.1 (FB)
- net +3.3VD: now also C10.1, C20.1, C8.1, C9.1, R14.1, R15.1, R33.1, R7.1, U1.2 (VDD), U6.6 (VDD), U6.7 (VREGIN)
- net +7V rectified: now reaches C30.1, C6.1, U5.1
- net +7V rectified: now also C25.1, D6.1 (A1), JP1.1 (A), U3.2 (EN), U3.3 (IN); no longer U2.2 (EN), U2.3 (IN)
- net at U6.26 (TXD): now also R26.1
- net at U6.25 (RXD): now also R28.1
- removed net +3.3V: C10.1, C11.1, C12.1, C20.1, C3.1, C8.1, C9.1, JP8.1 (A), JP9.3 (B), R14.1, R15.1, R33.1, R6.2, R7.1, U1.2 (VDD), U4.3 (DVDD), U6.6 (VDD), U6.7 (VREGIN)
- net 5V USB renamed +5V USB
- net +5V USB: now also JP1.3 (B)
- net CS: no longer names the net of U1.29 (IO5)
- net CS: now also R25.1; no longer U4.24 (~{CS})
- net MISO: no longer names the net of U4.26 (SDO/UTX)
- net MISO: now also R9.1; no longer U1.31 (IO19)
- net MOSI: no longer names the net of U1.37 (IO23)
- net MOSI: now also R10.1; no longer U4.27 (SDI/URX)
- net SCLK: no longer names the net of U1.30 (IO18)
- net SCLK: now also R13.1; no longer U4.25 (SCLK)
- net WarnOut renamed ATM_WO
- new net: C24.1, JP1.2 (C), U2.2 (EN), U2.3 (IN)
- new net: C31.1, C32.1, L2.2, U3.1 (FB), U7.1 (Vin), U7.2 (Vin), U7.3 (~{SHDN})
- new net: C26.1, U3.6 (BST)
- new net: C26.2, L2.1, U3.5 (SW)
- new net ATM_CS: R25.2, U4.24 (~{CS})
- new net ATM_SCLK: R13.2, U4.25 (SCLK)
- new net ATM_SDI: R10.2, U4.27 (SDI/URX)
- new net ATM_SDO: R9.2, U1.31 (IO19)
- no-connect marks 18 -> 19
Other:
- note added: "AGND i DGND treba da budu fizicki odvojeni ground planovi, spajaju se na jednoj tački direktno ispod čipa ili na ulazu napajanja"
- note added: "ATM90E26"
- note added: "AUTO PROGRAM"
- note added: "Alternative: AMS1117-3.3 MIC29302AWD"
- note added: "Alternativne opcije za buck su LM2596"
- note added: "BUTTONS"
- note added: "Biramo USB napajanje ili merni napon"
- note added: "DISPLAY"
- note added: "Low ESR Caps"
- note added: "MCU"
- note added: "Ovi 0R mogu da se zamene sa 33R ako bude potrebe"
- note added: "Ovi otpornici od 33R su tkz Series termination otpornici. Smanjuju sum, pogotovo kod dugackih traceova"
- note added: "POWER SUPPLY"
- note added: "Posto ce mcu da vuce mnogo struje, ovde je buck konvertor kako bi imali malu disipaciju"
- note added: "Pretvaramo 7V iz mernog u 5V koje ce posle LDO spustiti u 3.3V, ovo moramo jer je merni chip veoma osetljiv na sum"
- note added: "Proveriti da li ce u softveru biti potrebno da se ugasi SPI linija kada se utakne usb"
- note added: "TVS dioda za svaki slucaj"
- note added: "Tantalumski kondenzatori jer imaju malu serijsku otpornost sto je bitno za regulatore!"
- note added: "USB INTERFACE"
- note removed: "Alternativa AMS1117-3.3"
- note removed: "Alternativne opcije za buck su AP63205WU, koji daje 5V na izlazu, LM2596-5, koji isto daje 5V na izlazu."
- note removed: "Bilo bi dobro da se nadje verzija sa fiksnim izlaznim naponom a da nije preko 5 evra"
- note removed: "Moramo imati buck konvertor jer je jedini nacin da vucemo preko 1A, a da ne zapalimo LDO. Cilj je da 4V iz buck-a dovedemo na LDO koji ce izbaciti stabilnih 3.3V bez switching noise koji bi smetao mernom chipu"
- note removed: "Mozda nam ni ne treba LDO, moramo se dogovoriti, i dalje nisam siguran da li buck ima dovoljno mali noise"
- note removed: "Tantalumski kondenzatori jer imaju malu serijsku otpornost sto je bitno za ovaj regulator!"
- moved on the sheet: C1, C10, C11, C12, C13, C14, C15, C16, C17, C18, C19, C20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

Commit message: Displej, SD kartica, DigiKey modeli
Parts:
- removed JP1: Jumper_3_Open, symbol Jumper:Jumper_3_Open
- removed U3: AP63205WU, Package_TO_SOT_SMD:TSOT-23-6, symbol Regulator_Switching:AP63205WU
- added C2: 100n, symbol Device:C_Small
- added C33: 100p, symbol Device:C_Small
- added C34: 0.1u DNP, symbol Device:C_Small
- added H1: Jumper_Shunt, symbol Auxiliary_Items:Jumper_Shunt
- added J2: MEM2067-02-180-00-A, symbol Connector:Micro_SD_Card
- added J5: 541324062, CON_541324062_MOL, symbol Molex0541324062:541324062
- added J6: Conn_01x03_Pin, symbol Connector:Conn_01x03_Pin
- added R29: 157k, symbol Device:R_US
- added R30: 30k, symbol Device:R_US
- added R34, R8: 10k, symbol Device:R_US
- added SW3: SW_Push_2_Blue, symbol Switch:SW_Push
- added U3: AP63200WU, Package_TO_SOT_SMD:TSOT-23-6, symbol Regulator_Switching:AP63200WU
- C24, C25: value 10u Low ESR -> 10u X7R
- C3: value 22u Tant -> 10u X7R
- D2, D3, D4: DigiKey Part Number (none) -> ESD9B5.0ST5GOSCT-ND; MNF (none) -> onsemi; MPN (none) -> ESD9B5.0ST5G
- D5: value BAT760-7 -> BAT760; DigiKey Part Number (none) -> 5399-BAT760CT-ND; MNF (none) -> Shenzhen Slkormicro Semicon Co., Ltd.; MPN (none) -> BAT760
- D6: DigiKey Part Number (none) -> SMAJ12ALFCT-ND; MNF (none) -> Littelfuse Inc.; MPN (none) -> SMAJ12A
- J1: DigiKey Part Number (none) -> 2073-USB4125-GF-A-0190CT-ND; MNF (none) -> GCT; MPN (none) -> USB4125-GF-A-0190
- J3: DigiKey Part Number (none) -> CP-002AHPJCT-ND; MNF (none) -> Same Sky (Formerly CUI Devices); MPN (none) -> PJ-002AH-SMT-TR
- J4: DigiKey Part Number (none) -> CP-3523SJCT-ND; MNF (none) -> Same Sky (Formerly CUI Devices); MPN (none) -> SJ-3523-SMT-TR
- L2: value 4.7u -> 10u
- Q1, Q2: DigiKey Part Number (none) -> 5399-SS8050CT-ND; MNF (none) -> Shenzhen Slkormicro Semicon Co., Ltd.; MPN (none) -> SS8050
- SW1, SW2: value SW_Push -> SW_Push_1_Red; DigiKey Part Number (none) -> CKN9084CT-ND; MNF (none) -> C&K; MPN (none) -> PTS645SK43SMTR92 LFS
- U1: value ESP32-WROOM-32E -> ESP32-WROOM-32E-N4; DigiKey Part Number (none) -> 1965-ESP32-WROOM-32E-N4CT-ND; MNF (none) -> Espressif Systems; MPN (none) -> ESP32-WROOM-32E-N4
- U2: DigiKey Part Number (none) -> AP63203WU-7DICT-ND; MNF (none) -> Diodes Incorporated; MPN (none) -> AP63203WU-7
- U4: DigiKey Part Number (none) -> ATM90E26-YU-RCT-ND; MNF (none) -> Microchip Technology; MPN (none) -> ATM90E26-YU-R
- U5: MNF (none) -> ABS210-13DICT-ND; MPN (none) -> ABS210-13
- U6: value CP2102N-A02-GQFN28 -> CP2102N-A02-GQFN28R; DigiKey Part Number (none) -> 336-5890-1-ND; MNF (none) -> Silicon Labs; MPN (none) -> CP2102N-A02-GQFN28R
- U7: value MCP1727-3302xSN -> MCP1727-3302E/SN; DigiKey Part Number (none) -> MCP1727T-3302E/SNCT-ND; MNF (none) -> Microchip Technology; MPN (none) -> MCP1727T-3302E/SN
- Y1: value 8.192MHz -> ABLS-8.192MHZ-B2-T; footprint (none) -> Crystal:Crystal_SMD_HC49-SD; DigiKey Part Number (none) -> 535-9090-1-ND; MNF (none) -> Abracon LLC; MPN (none) -> ABLS-8.192MHZ-B2-T
Connections:
- net +3.3VD: now also C2.1, J2.4 (VDD), J5.12, J5.13, J5.14, J5.15, J5.16, J5.17, J5.18, J5.19, J5.20, J5.21, J5.22, J5.23, J5.24, J5.25, J5.26, J5.27, J5.28, J5.29, J5.31, J5.32, J5.38, J5.7, J5.8, R34.1, R8.1
- net +7V rectified: now also J6.3 (Pin_3), U3.2 (EN), U3.3 (IN)
- net GND: now also C2.2, C34.2, J2.6 (VSS), J5.1, J5.33, J5.34, J5.35, J5.36, J5.37, J5.39, R30.2, SW3.2, U3.4 (GND)
- net VBUS: now also J6.1 (Pin_1)
- net at C24.1, U2.2 (EN), U2.3 (IN): now also J6.2 (Pin_2)
- net at C31.1, C32.1, L2.2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: now also C33.1, R29.1
- net at C26.1: now also U3.6 (BST)
- net at C26.2, L2.1: now also U3.5 (SW)
- net +5V USB renamed +5V_EXT
- new net: C33.2, R29.2, R30.1, U3.1 (FB)
- new net BT: C34.1, R34.2, SW3.1
- new net DSP_CS: J5.10
- new net DSP_RESX: J5.30
- new net DSP_SCLK: J5.11
- new net DSP_SDI: J5.9
- new net DSP_SDO: J5.6
- new net DSP_TE: J5.40
- new net SD_CS: J2.2 (DAT3/CD), R8.2
- new net SD_SCLK: J2.5 (CLK)
- new net SD_SDI: J2.3 (CMD)
- new net SD_SDO: J2.7 (DAT0)
- no-connect marks 19 -> 28
Other:
- note added: "DISPLAY I SD"
- note added: "Displej konektor"
- note added: "https://forum.arduino.cc/t/micro-sd-card-module-schematics/1341510"
- note added: "https://newhavendisplay.com/content/specs/NHD-2.4-240320AF-CSXP.pdf"
- note added: "mozda na gnd"
- note removed: "DISPLAY"
- note removed: "Tantalumski kondenzatori jer imaju malu serijsku otpornost sto je bitno za regulatore!"
- moved on the sheet: C1, C31, C32, C4, C5, R14, R15, SW1

Commit message: Power MUX, Display, Part numbers, Manufacturers and Footprints
Parts:
- removed C1, C15: 1u, symbol Device:C_Small
- removed C12, C13: 0.1u, symbol Device:C_Small
- removed C14, C21: 33n, symbol Device:C_Small
- removed C2, C7: 100n, symbol Device:C_Small
- removed C20: 0.1u/50V, symbol Device:C
- removed C23: 12p, symbol Device:C_Small
- removed C24, C25, C3: 10u X7R, symbol Device:C_Polarized
- removed C27: 1uF/16V(10%), symbol Device:C
- removed C28, C29, C31, C32, C9: 22u, symbol Device:C_Polarized
- removed C4, C5: 0.1u DNP, symbol Device:C_Small
- removed C6: 470u Low ESR Electr, symbol Device:C_Polarized
- removed C8: 100n/50V 10%, symbol Device:C_Small
- removed H1: Jumper_Shunt, symbol Auxiliary_Items:Jumper_Shunt
- removed J6: Conn_01x03_Pin, symbol Connector:Conn_01x03_Pin
- removed JP8, JP9: 2+3, symbol Jumper:SolderJumper_3_Open
- removed R1: 2k, symbol Device:R_US
- removed R10, R13, R9: 33R, symbol Device:R_Small_US
- removed R11, R12: 10k 5%, symbol Device:R_US
- removed R14, R15: 10k, symbol Device:R_US
- removed R27: 4k2, symbol Device:R_US
- removed R3: 5k1, symbol Device:R_US
- removed R6: 0, symbol Device:R_US
- added C1, C2, C3: 10u, Capacitor_SMD:C_0805_2012Metric, symbol Device:C
- added C12, C4, C5, C6, C8: 22u, Capacitor_SMD:C_1210_3225Metric, symbol Device:C
- added C27: 1u, Capacitor_SMD:C_0603_1608Metric, symbol Device:C_Small
- added C35, C38, C39, C42, C44, C45, C47, C48, C49, C50, C51: 100n, Capacitor_SMD:C_0603_1608Metric, symbol Device:C_Small
- added C36, C41: 33n, Capacitor_SMD:C_0603_1608Metric, symbol Device:C_Small
- added C37: 4.7m, Capacitor_SMD:CP_Elec_16x22, symbol Device:C_Polarized
- added C40: 12p, Capacitor_SMD:C_0603_1608Metric, symbol Device:C_Small
- added D8: LED_BLUE, LED_SMD:LED_0805_2012Metric, symbol Device:LED
- added D9: LED_ORANGE, LED_SMD:LED_0805_2012Metric, symbol Device:LED
- added JP1, JP2: 2+1, symbol Jumper:SolderJumper_3_Bridged12
- added R1, R3: 10k, Resistor_SMD:R_0603_1608Metric, symbol Device:R_Small_US
- added R10, R9: 330R, Resistor_SMD:R_0603_1608Metric, symbol Device:R_US
- added R35: 0R, Resistor_SMD:R_0603_1608Metric, symbol Device:R_Small_US
- added R36, R38, R39, R40, R41, R46, R48, R49, R50: 33R, Resistor_SMD:R_0603_1608Metric, symbol Device:R_Small_US
- added R37, R45, R51, R53, R54, R56, R57, R58: 10k, Resistor_SMD:R_0603_1608Metric, symbol Device:R_US
- added R44: 21k5, Resistor_SMD:R_0603_1608Metric, symbol Device:R_Small_US
- added R55, R59: 18k2, Resistor_SMD:R_0603_1608Metric, symbol Device:R_Small_US
- added U8: TPS2121RUXR, RUX0012A, symbol TPS2121RUXR:TPS2121RUXR
- added U9: NHD-2.4-240320AF-CSXP, Display:EA_eDIPTFT32-XXX, symbol Display_Graphic:EA_eDIPTFT32-A
- C10: value 4u7/6V3 -> 4u7; footprint (none) -> Capacitor_SMD:C_0603_1608Metric; DigiKey Part Number (none) -> 490-7203-1-ND; MNF (none) -> Murata Electronics; MPN (none) -> GRM188R61E475KE11D
- C11: value 47u Elec -> 47u; footprint (none) -> Capacitor_SMD:CP_Elec_6.3x5.2; DigiKey Part Number (none) -> 565-EMVE250ARA470MF55GCT-ND; MNF (none) -> Chemi-Con; MPN (none) -> EMVE250ARA470MF55G
- C16: footprint (none) -> Capacitor_SMD:C_0603_1608Metric; DigiKey Part Number (none) -> 399-C0603C102K5RACTUCT-ND; MNF (none) -> KEMET; MPN (none) -> C0603C102K5RACTU
- C17: value 0.1u -> 1u; footprint (none) -> Capacitor_SMD:C_0603_1608Metric; DigiKey Part Number (none) -> 399-C0603C105K4RACTUCT-ND; MNF (none) -> KEMET; MPN (none) -> C0603C105K4RACTU
- C18, C19: footprint (none) -> Capacitor_SMD:C_0603_1608Metric; DigiKey Part Number (none) -> 445-5950-1-ND; MNF (none) -> TDK; MPN (none) -> C1608X7R1H334K080AC
- C22: footprint (none) -> Capacitor_SMD:C_0603_1608Metric; DigiKey Part Number (none) -> 478-KGQ15ACG2D120GTCT-ND; MNF (none) -> KYOCERA AVX; MPN (none) -> KGQ15ACG2D120GT
- C26: value 100n -> 1u; footprint (none) -> Capacitor_SMD:C_0603_1608Metric; DigiKey Part Number (none) -> 399-C0603C105K4RACTUCT-ND; MNF (none) -> KEMET; MPN (none) -> C0603C105K4RACTU
- C30: footprint (none) -> Capacitor_SMD:C_0603_1608Metric; DigiKey Part Number (none) -> 399-C0603C104K3RACTUCT-ND; MNF (none) -> KEMET; MPN (none) -> C0603C104K3RACTU
- C33: footprint (none) -> Capacitor_SMD:C_0603_1608Metric; DigiKey Part Number (none) -> 490-1427-1-ND; MNF (none) -> Murata Electronics; MPN (none) -> GRM1885C1H101JA01D
- C34: value 0.1u DNP -> 100n; footprint (none) -> Capacitor_SMD:C_0603_1608Metric; DigiKey Part Number (none) -> 399-C0603C104K3RACTUCT-ND; MNF (none) -> KEMET; MPN (none) -> C0603C104K3RACTU
- D1: footprint (none) -> LED_SMD:LED_0805_2012Metric; DigiKey Part Number (none) -> 160-1426-1-ND; MNF (none) -> Lite-On Inc.; MPN (none) -> LTST-C171KGKT
- D7: footprint (none) -> LED_SMD:LED_0805_2012Metric; DigiKey Part Number (none) -> 160-1427-1-ND; MNF (none) -> Lite-On Inc.; MPN (none) -> LTST-C171KRKT
- L1: value 3.9u -> 4u7; footprint (none) -> Inductor_SMD:L_1210_3225Metric; DigiKey Part Number (none) -> 490-10594-1-ND; MNF (none) -> Murata Electronics; MPN (none) -> 1277AS-H-4R7M=P2
- L2: footprint (none) -> Inductor_SMD:L_1210_3225Metric; DigiKey Part Number (none) -> 535-AOTA-C322512Q100MTCT-ND; MNF (none) -> Abracon LLC; MPN (none) -> AOTA-C322512Q100MT
- R16: value 4k2 -> 4k22; footprint (none) -> Resistor_SMD:R_0603_1608Metric; DigiKey Part Number (none) -> 311-4.22KHRCT-ND; MNF (none) -> YAGEO; MPN (none) -> RC0603FR-074K22L
- R17, R18: footprint (none) -> Resistor_SMD:R_0603_1608Metric; DigiKey Part Number (none) -> 311-3.00KHRCT-ND; MNF (none) -> YAGEO; MPN (none) -> RC0603FR-073KL
- R19, R20: value 100 -> 100R; footprint (none) -> Resistor_SMD:R_0603_1608Metric; DigiKey Part Number (none) -> 311-100HRCT-ND; MNF (none) -> YAGEO; MPN (none) -> RC0603FR-07100RL
- R2: footprint (none) -> Resistor_SMD:R_0201_0603Metric; DigiKey Part Number (none) -> 311-1MMCT-ND; MNF (none) -> YAGEO; MPN (none) -> RC0201FR-071ML
- R21: value 5.3k -> 4k22; footprint (none) -> Resistor_SMD:R_0603_1608Metric; DigiKey Part Number (none) -> 311-4.22KHRCT-ND; MNF (none) -> YAGEO; MPN (none) -> RC0603FR-074K22L
- R22, R23: value 5.3k -> 7k87; footprint (none) -> Resistor_SMD:R_0603_1608Metric; DigiKey Part Number (none) -> 311-7.87KHRCT-ND; MNF (none) -> YAGEO; MPN (none) -> RC0603FR-077K87L
- R24: footprint (none) -> Resistor_SMD:R_0603_1608Metric; DigiKey Part Number (none) -> 311-1.00KHRCT-ND; MNF (none) -> YAGEO; MPN (none) -> RC0603FR-071KL
- R25: footprint (none) -> Resistor_SMD:R_0603_1608Metric; DigiKey Part Number (none) -> 13-RC0603FR-0733RLCT-ND; MNF (none) -> YAGEO; MPN (none) -> RC0603FR-0733RL
- R26, R28: footprint (none) -> Resistor_SMD:R_0603_1608Metric; DigiKey Part Number (none) -> 311-0.0GRCT-ND; MNF (none) -> YAGEO; MPN (none) -> RC0603JR-070RL
- R29: value 157k -> 158k; footprint (none) -> Resistor_SMD:R_0603_1608Metric; DigiKey Part Number (none) -> 311-158KHRCT-ND; MNF (none) -> YAGEO; MPN (none) -> RC0603FR-07158KL
- R30: footprint (none) -> Resistor_SMD:R_0603_1608Metric; DigiKey Part Number (none) -> 311-30.0KHRCT-ND; MNF (none) -> YAGEO; MPN (none) -> RC0603FR-0730KL
- R31: value 22k1 1% -> 22k1; footprint (none) -> Resistor_SMD:R_0603_1608Metric; DigiKey Part Number (none) -> 311-22.1KHRCT-ND; MNF (none) -> YAGEO; MPN (none) -> RC0603FR-0722K1L
- R32: value 47k5 1% -> 47k5; footprint (none) -> Resistor_SMD:R_0603_1608Metric; DigiKey Part Number (none) -> 13-RC0603FR-1047K5LCT-ND; MNF (none) -> YAGEO; MPN (none) -> RC0603FR-1047K5L
- R33: value 2k (5%) -> 2k; footprint (none) -> Resistor_SMD:R_0603_1608Metric; DigiKey Part Number (none) -> 311-2.00KHRCT-ND; MNF (none) -> YAGEO; MPN (none) -> RC0603FR-072KL
- R34: value 10k -> 1k; footprint (none) -> Resistor_SMD:R_0603_1608Metric; DigiKey Part Number (none) -> 311-1.00KHRCT-ND; MNF (none) -> YAGEO; MPN (none) -> RC0603FR-071KL
- R4: footprint (none) -> Resistor_SMD:R_0603_1608Metric; DigiKey Part Number (none) -> 311-5.10KHRCT-ND; MNF (none) -> YAGEO; MPN (none) -> RC0603FR-075K1L
- R5: value 1k -> 5k1; footprint (none) -> Resistor_SMD:R_0603_1608Metric; DigiKey Part Number (none) -> 311-5.10KHRCT-ND; MNF (none) -> YAGEO; MPN (none) -> RC0603FR-075K1L
- R7: value 2k -> 330R; footprint (none) -> Resistor_SMD:R_0603_1608Metric; DigiKey Part Number (none) -> 311-330HRCT-ND; MNF (none) -> YAGEO; MPN (none) -> RC0603FR-07330RL
- R8: value 10k -> 330R; footprint (none) -> Resistor_SMD:R_0603_1608Metric; DigiKey Part Number (none) -> 311-330HRCT-ND; MNF (none) -> YAGEO; MPN (none) -> RC0603FR-07330RL
- TP1, TP2, TP3, TP6: now left out of the parts list
- U5: DigiKey Part Number (none) -> ABS210-13DICT-ND; MNF ABS210-13DICT-ND -> Diodes Incorporated
Connections:
- net DSP_SCLK is gone; now on net SCLK: J5.11
- net DSP_SDI is gone; now on net MOSI: J5.9
- net +3.3VA: now also R8.1, C2.1, C38.2, JP1.3 (B), JP2.1 (A), R35.2
- net +3.3VD: now also C12.1, C45.2, C50.1, C51.2, C6.1, C8.1, R37.2, R45.2, R53.2, R54.1, R56.2, R58.2; no longer R34.1, R8.1
- net +7V rectified: now also C37.1, R55.1, U8.7 (IN1); no longer U3.2 (EN), U3.3 (IN)
- net ATM_CS: now also R53.1
- net ATM_IRQ: now also U1.10 (IO25); no longer U1.13 (IO14)
- net ATM_WO: now also U1.11 (IO26); no longer U1.14 (IO12)
- net BT: now also C49.2, R56.1; no longer C34.1, R34.2
- net DSP_CS: now also R41.2, R54.2
- net DSP_RESX: now also U1.27 (IO16)
- net DSP_TE: now also U1.28 (IO17)
- net DTR: now also R51.2
- net EN: now also C27.1, C47.2, R37.1
- net GND: now also C17.2, C26.2, C34.1, R34.1, U4. (RESV_LOW), C1.2, C12.2, C2.2, C27.2, C3.2, C36.2, C37.2, C38.1, C39.1, C4.2, C40.1, C41.2, C44.1, C45.1, C47.1, C48.1, C49.1, C5.2, C50.2, C51.1, C6.2, C8.2, D8.1 (K), D9.1 (K), JP1.1 (A), JP2.3 (B), R1.2, R3.2, R44.2, U8.12 (GND), U8.4 (OV2), U8.5 (OV1), U8.9 (ST); no longer C17.1, C34.2
- net IO0: now also C48.2, R45.1
- net N: now also R22.2; no longer R21.1
- net RTS: now also R57.2
- net SD_CS: now also R40.2, R58.1; no longer R8.2
- net SD_SCLK: now also R38.2
- net VBUS: now also C17.1, R59.1, U8.2 (IN2)
- net VP: now also R23.1, C41.1; no longer R23.2
- net at U4.15 (VN): now also R34.2, C36.1; no longer R5.1
- net at R18.2, R20.1: now also R21.2
- net V_IN: now reaches U2.2 (EN), U2.3 (IN)
- net V_IN: now also U3.2 (EN), U3.3 (IN), C1.1, C3.1, U8.1 (OUT), U8.8 (OUT)
- net at L1.1, U2.5 (SW): now also C42.2
- net at U2.6 (BST): now also C42.1
- net at L2.1, U3.5 (SW): now also C35.2; no longer C26.2
- net at U3.6 (BST): now also C35.1; no longer C26.1
- net at C33.1, L2.2, R29.1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: now also C4.1, C5.1
- net at U4.5 (AVDD): now also C44.2, R35.1
- net at J4.1 (SLEEVE): now also R21.1
- net at Q1.1 (B): now also R51.1
- net at C16.1, TP6.1, U4.13 (Vref): now also C26.1
- net at U4.1 (MMD1): now also JP1.2 (C)
- net at J1.A5 (CC1): now also R5.1
- net at U1.16 (IO13): now also R36.1
- net at U1.23 (IO15): now also R40.1
- net random: now reaches U1.26 (IO4)
- net random: now also R10.1
- net at U1.30 (IO18): now also R46.1
- net at U1.33 (IO21): now also R41.1
- net BT_LED: now reaches U1.36 (IO22)
- net BT_LED: now also R9.1
- net at U1.37 (IO23): now also R48.1
- net at U4.22 (OSCI), Y1.1: now also C40.2
- net at U4.4 (~{Reset}): now also C39.2; no longer C17.2
- net at Q2.1 (B): now also R57.1
- net at U4.28 (MMD0): now also JP2.2 (C)
- net at U4.26 (SDO/UTX): now also R39.1
- net at D1.2 (A): now also R8.2
- net at R22.1: now also R23.2; no longer R23.1
- net ATM_SCLK renamed SCLK
- net SCLK: now also R46.2
- net ATM_SDI renamed MOSI
- net MOSI: now also R48.2
- net ATM_SDO renamed MISO
- net MISO: now also R39.2, R50.1
- net DSP_SDO: no longer names the net of J5.6
- net DSP_SDO: now also R50.2
- net SD_SDI renamed SD_MOSI
- net SD_MOSI: now also R36.2
- net SD_SDO: no longer names the net of J2.7 (DAT0)
- net SD_SDO: now also R49.2
- new net: D8.2 (A), R9.2
- new net: R1.1, R59.2, U8.3 (CP2)
- new net: C34.2, U8.11 (SS)
- new net: R44.1, U8.10 (ILM)
- new net: D9.2 (A), R10.2
- new net: R38.1, U1.13 (IO14)
- new net: R3.1, R55.2, U8.6 (PR1)
- new net SD_MISO: R49.1, U1.14 (IO12)
- no-connect marks 28 -> 73
Other:
- note added: "Ostavio sam sve pinove na displayu nepovezane jer svakako idu na konektor, o vaj displej je vise placeholder za BOM, pravi displey nece biti deo PCB-a"
- note added: "Ovde proveriti da li uopste zelimo otpornike (vise je safe ali mozda je nepotrebno)"
- note added: "Softverski pogasiti sve kad PROG, ekran dimmovati"
- note added: "proveri footprint"
- note removed: "Low ESR Caps"
- moved on the sheet: C22, C33, D1, D6, J2, J3, J5, L2, R29, R30, R7, U3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

Commit message: Displej napajanje reseno (valjda)
Parts:
- removed R23: 7k87, Resistor_SMD:R_0603_1608Metric, symbol Device:R_US
- added Q3: AO3400A, Package_TO_SOT_SMD:SOT-23, symbol Transistor_FET:AO3400A
- added R11, R6: 40R, symbol Device:R_Small_US
- added R60, R61, R62, R63: 10k, Resistor_SMD:R_0603_1608Metric, symbol Device:R_US
- C11: value 47u -> 10u promeni mnp, mora elec
- R22: value 7k87 -> 100R; DigiKey Part Number 311-7.87KHRCT-ND -> 311-100HRCT-ND; MPN RC0603FR-077K87L -> RC0603FR-07100RL
- R44: value 21k5 -> 82k; footprint Resistor_SMD:R_0603_1608Metric -> (none); DigiKey Part Number 311-21.5KHRCT-ND -> (none); MNF YAGEO -> (none); MPN RC0603FR-0721K5L -> (none)
Connections:
- net +3.3VD: now also R63.1; no longer J5.38
- net GND: now also J5.P1, J5.P2, Q3.2 (S), R62.2; no longer J5.34, J5.35, J5.36, J5.37
- net N: now also R60.2; no longer R22.2
- net VP: now also R61.1
- net +5V: now reaches C33.1, C4.1, C5.1, L2.2, R29.1, U7.1 (Vin), U7.2 (Vin), U7.3 (~{SHDN})
- net +5V: now also R11.2, R6.2
- net DSP_BRIGHT: now reaches U1.24 (IO2)
- net DSP_BRIGHT: now also R22.1
- new net: Q3.1 (G), R22.2, R62.1
- new net: R60.1, R61.2
- new net LED-A: J5.38, R11.1, R6.1
- new net LED-K1: J5.34, J5.35, J5.36, J5.37, Q3.3 (D), R63.2
- no-connect marks 73 -> 70
Other:
- note added: "0.2W res"
- note added: "mnp"
- note removed: "Softverski pogasiti sve kad PROG, ekran dimmovati"
- note removed: "mozda na gnd"
- moved on the sheet: J5, R50, R54
