File: project_files/Ohmsprint.kicad_sch (KiCad schematic)
At the start: 126 parts, among them J1 USB_C_Receptacle_USB2.0_16P, J2 MEM2067-02-180-00-A, J3 PJ-002AH-SMT-TR, J4 SJ-3523-SMT-TR, J5 541324062, Q1 SS8050, Q2 SS8050, Q3 AO3400A, SW1 SW_Push_1_Red, SW2 SW_Push_1_Red, SW3 SW_Push_2_Blue, U1 ESP32-WROOM-32E-N4, U2 AP63203WU, U3 AP63200WU, U4 ATM90E26-YU, U5 ABS210-13, U6 CP2102N-A02-GQFN28R, U7 MCP1727-3302E/SN, U8 TPS2121RUXR, U9 NHD-2.4-240320AF-CSXP, Y1 ABLS-8.192MHZ-B2-T

Commit message: Generisan Bill of Materials
Parts:
- added R12: 56k, Resistor_SMD:R_0603_1608Metric, symbol Device:R_US
- added R13: 40R2, Resistor_SMD:R_0805_2012Metric, symbol Device:R_Small_US
- added R14, R23: 20R, Resistor_SMD:R_0805_2012Metric, symbol Device:R_Small_US
- added R15: 10R, Resistor_SMD:R_0805_2012Metric, symbol Device:R_Small_US
- added R42: 22k1, Resistor_SMD:R_0603_1608Metric, symbol Device:R_US
- added R64: 10k, Resistor_SMD:R_0603_1608Metric, symbol Device:R_US
- C11: value 10u promeni mnp, mora elec -> 10u; footprint Capacitor_SMD:CP_Elec_6.3x5.2 -> Capacitor_SMD:CP_Elec_4x5.7; DigiKey Part Number 565-EMVE250ARA470MF55GCT-ND -> 399-17336-1-ND; MNF Chemi-Con -> KEMET; MPN EMVE250ARA470MF55G -> EDH106M016A9BAA
- Q3: DigiKey Part Number (none) -> 4518-AO3400ACT-ND; MNF (none) -> UMW; MPN (none) -> AO3400A
- R11: value 40R -> 40R2; footprint (none) -> Resistor_SMD:R_0805_2012Metric; DigiKey Part Number (none) -> 541-40.2CCT-ND; MNF (none) -> Vishay Dale; MPN (none) -> CRCW080540R2FKEA
- R44: value 82k -> 82k5; footprint (none) -> Resistor_SMD:R_0805_2012Metric; DigiKey Part Number (none) -> RMCF0805FT82K5CT-ND; MNF (none) -> Stackpole Electronics Inc; MPN (none) -> RMCF0805FT82K5
- R6: value 40R -> 10R; footprint (none) -> Resistor_SMD:R_0805_2012Metric; DigiKey Part Number (none) -> 541-10ACT-ND; MNF (none) -> Vishay Dale; MPN (none) -> CRCW080510R0JNEA
Connections:
- net +5V: now also R13.2; no longer R6.2
- net LED-A: now also R13.1; no longer R6.1
- no-connect marks 70 -> 84
Other:
- note added: "pulldown za gpio12"
- note removed: "0.2W res"
- note removed: "mnp"

Commit message: USB :)
Parts:
- removed D3, D4: ESD9B5.0ST5G, Diode_SMD:D_SOD-923, symbol Diode:ESD9B5.0ST5G
- removed J1: USB_C_Receptacle_USB2.0_16P, symbol Connector:USB_C_Receptacle_USB2.0_16P
- removed R2: 1M, Resistor_SMD:R_0201_0603Metric, symbol Device:R_US
- removed R4, R5: 5k1, Resistor_SMD:R_0603_1608Metric, symbol Device:R_US
- removed R40: 33R, Resistor_SMD:R_0603_1608Metric, symbol Device:R_Small_US
- added D10, D11: ESD9B5.0ST5G, Diode_SMD:D_SOD-923, symbol Diode:ESD9B5.0ST5G
- added J6: USB4110-GF-A, USB4110-GF-A_GCT, symbol USB4110-GF-A:USB4110-GF-A
- added R27, R40: 5k1, Resistor_SMD:R_0603_1608Metric, symbol Device:R_US
- added R52: 33R, Resistor_SMD:R_0603_1608Metric, symbol Device:R_Small_US
- added TP4: TestPoint, symbol Connector:TestPoint
Connections:
- net ATIM_CF1: no longer U1.9 (IO33)
- net ATM_IRQ: now also U1.7 (IO35); no longer U1.10 (IO25)
- net ATM_ZX: now also U1.8 (IO32); no longer U1.12 (IO27)
- net DSP_BRIGHT: now also U1.9 (IO33); no longer U1.24 (IO2)
- net GND: now also D10.1 (A1), D11.1 (A1), J6.A1-B12 (GND), J6.A12-B1 (GND), R27.2, R40.1
- net IO0: now also TP4.1
- net SD_CS: now also R52.2
- net SD_MISO: now also U1.11 (IO26); no longer U1.14 (IO12)
- net VBUS: now also J6.A4-B9 (VBUS), J6.A9-B4 (VBUS)
- net ATM_CF1: now reaches U1.6 (IO34)
- net ATM_CF2: no longer names the net of U4.19 (CF2)
- net ATM_CF2: no longer U1.8 (IO32)
- net ATM_WO: no longer names the net of U4.17 (WarnOut)
- net ATM_WO: no longer U1.11 (IO26)
- new net: R52.1, U1.12 (IO27)
- new net: J6.A5 (CC1), R40.2
- new net: J6.B5 (CC2), R27.1
- new net D+: D10.2 (A2), J6.A6 (DP1), J6.B6 (DP2)
- new net D-: D11.2 (A2), J6.A7 (DN1), J6.B7 (DN2)
- no-connect marks 84 -> 88
Other:
- note removed: "Ovde proveriti da li uopste zelimo otpornike (vise je safe ali mozda je nepotrebno)"

Commit message: Uradjeno pola rutiranja
Parts:
- removed D5: BAT760, symbol Device:D_Schottky
- removed R35: 0R, Resistor_SMD:R_0603_1608Metric, symbol Device:R_Small_US
- added R35: 0R, symbol Device:R_US
- C37: footprint Capacitor_SMD:CP_Elec_16x22 -> Capacitor_SMD:CP_Elec_16x17.5
- J2: footprint (none) -> usb:CONN_MEM2067-02-180-00-A_GCT
- J3: footprint PJ-002AH-SMT-TR:CUI_PJ-002AH-SMT-TR -> PJ_002AH:PJ-002AH-SMT-TR_CUD
- J4: footprint SJ-3523-SMT-TR:CUI_SJ-3523-SMT-TR -> SJ_3523_SMT:SJ-3523-SMT_CUD
- J5: footprint CON_541324062_MOL -> 541324062:CON_541324062_MOL
- J6: footprint USB4110-GF-A_GCT -> USB4110-GF-A-foot:USB4110-GF-A_GCT
- JP1, JP2: footprint (none) -> Jumper:SolderJumper-3_P1.3mm_Bridged12_RoundedPad1.0x1.5mm
- SW1, SW2: footprint (none) -> red:SWITCH_45SK43SMTR92LFS
- SW3: footprint (none) -> blue:SWITCH_43SMTR92LFS
- TP1, TP2, TP3, TP4, TP6: footprint (none) -> test_points:TestPoint_Pad_D2.0mm
- U1: footprint RF_Module:ESP32-WROOM-32D -> esp32_custom:ESP32-WROOM-32D
- U5: footprint SON_S210-13_DIO -> ABS210-13:SON_S210-13_DIO
- U6: footprint QFN28_5X5_SIL -> cp2102n-a02-gqfn28-foot:QFN28_5X5_SIL
- U8: footprint RUX0012A -> TPS2121RUXR:RUX0012A
Connections:
- net +3.3VA: now also C44.2, U4.5 (AVDD); no longer C11.1, C38.2, U4.3 (DVDD)
- net +3.3VD: now also C11.1, C38.2, U4.3 (DVDD)
- net GND: now also R35.1; no longer C16.2, C18.2, C19.1, C26.2, C36.2, C41.2, C44.1, R17.2, R18.1, R24.1, R34.1, U4.14 (AGND), U4.6 (AGND), U4.7 (I2P), U4.8 (I2N)
- new net GNDA: C16.2, C18.2, C19.1, C26.2, C36.2, C41.2, C44.1, R17.2, R18.1, R24.1, R34.1, R35.2, U4.14 (AGND), U4.6 (AGND), U4.7 (I2P), U4.8 (I2N)
