File: project_files/Ohmsprint.kicad_sch (KiCad schematic)
At the start: 132 parts, among them J2 MEM2067-02-180-00-A, J3 PJ-002AH-SMT-TR, J4 SJ-3523-SMT-TR, J5 541324062, J6 USB4110-GF-A, Q1 SS8050, Q2 SS8050, Q3 AO3400A, SW1 SW_Push_1_Red, SW2 SW_Push_1_Red, SW3 SW_Push_2_Blue, U1 ESP32-WROOM-32E-N4, U2 AP63203WU, U3 AP63200WU, U4 ATM90E26-YU, U5 ABS210-13, U6 CP2102N-A02-GQFN28R, U7 MCP1727-3302E/SN, U8 TPS2121RUXR, U9 NHD-2.4-240320AF-CSXP, Y1 ABLS-8.192MHZ-B2-T

Commit message: Uradjen PCB
Parts:
- removed D9: LED_ORANGE, LED_SMD:LED_0805_2012Metric, symbol Device:LED
- removed R10: 330R, Resistor_SMD:R_0603_1608Metric, symbol Device:R_US
- removed R12: 56k, Resistor_SMD:R_0603_1608Metric, symbol Device:R_US
- removed R14, R23: 20R, Resistor_SMD:R_0805_2012Metric, symbol Device:R_Small_US
- removed R15, R6: 10R, Resistor_SMD:R_0805_2012Metric, symbol Device:R_Small_US
- removed R35: 0R, symbol Device:R_US
- removed R42: 22k1, Resistor_SMD:R_0603_1608Metric, symbol Device:R_US
- removed R53, R58, R64: 10k, Resistor_SMD:R_0603_1608Metric, symbol Device:R_US
- added R43, R47, R65: 33R, Resistor_SMD:R_0603_1608Metric, symbol Device:R_Small_US
Connections:
- net Data+ is gone; now on net D+: U6.4 (D+)
- net Data- is gone; now on net D-: U6.5 (D-)
- net GNDA is gone; now on net GND: C16.2, C18.2, C19.1, C26.2, C36.2, C41.2, C44.1, R17.2, R18.1, R24.1, R34.1, U4.14 (AGND), U4.6 (AGND), U4.7 (I2P), U4.8 (I2N)
- net ATM_CF1: now also R65.2
- net ATM_IRQ: now also R47.2; no longer U4.20 (IRQ)
- net ATM_ZX: now also R43.2; no longer U4.21 (ZX)
- net ATIM_CF1: no longer names the net of U4.18 (CF1)
- net ATIM_CF1: now also R65.1
- net random: no longer names the net of U1.26 (IO4)
- new net: R43.1, U4.21 (ZX)
- new net: R47.1, U4.20 (IRQ)
- no-connect marks 88 -> 75
Other:
- note removed: "pulldown za gpio12"

Commit message: Generisani Gerber i Drill
Parts:
- removed J2: MEM2067-02-180-00-A, usb:CONN_MEM2067-02-180-00-A_GCT, symbol Connector:Micro_SD_Card
- added J1: MEM2067-02-180-00-A_REVB, MEM2067-02-180-00-A_REVB_foot:GCT_MEM2067-02-180-00-A_REVB, symbol MEM2067-02-180-00-A_REVB:MEM2067-02-180-00-A_REVB
- J3: footprint PJ_002AH:PJ-002AH-SMT-TR_CUD -> CUI_PJ-002AH-SMT-TR-foot:CUI_PJ-002AH-SMT-TR
- J4: footprint SJ_3523_SMT:SJ-3523-SMT_CUD -> CUI_SJ-3523-SMT-TR-foot:CUI_SJ-3523-SMT-TR
- J5: footprint 541324062:CON_541324062_MOL -> Molex0541324062-foot:CON_541324062_MOL
- U1: footprint esp32_custom:ESP32-WROOM-32D -> RF_Module:ESP32-WROOM-32D
- U8: footprint TPS2121RUXR:RUX0012A -> TPS2121RUXR-foot:RUX0012A
Connections:
- net +3.3VD: now also J1.4 (VDD)
- net GND: now also J1.6 (VSS)
- net SD_CS: now also J1.2 (CD/DAT3)
- net SD_MOSI: now also J1.3 (CMD)
- net SD_SCLK: now also J1.5 (CLK)
- net at R49.2: now also J1.7 (DAT0)
- new net: J1.10 (SHIELD), J1.11 (SHIELD), J1.12 (SHIELD), J1.9 (SHIELD)
