File: project_files/Ohmsprint.kicad_pcb (KiCad board)
At the start: 2 copper layers, 150 x 150 mm, 132 parts, among them J1 USB_C_Receptacle_USB2.0_16P, J2 MEM2067-02-180-00-A, J3 PJ-002AH-SMT-TR, J4 SJ-3523-SMT-TR, J5 541324062, Q1 SS8050, Q2 SS8050, Q3 AO3400A, SW1 SW_Push_1_Red, SW2 SW_Push_1_Red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

Commit message: USB :)
Parts:
- removed D3, D4: ESD9B5.0ST5G, Diode_SMD:D_SOD-923
- removed J1: USB_C_Receptacle_USB2.0_16P, usb:CONN_MEM2067-02-180-00-A_GCT
- removed R2: 1M, Resistor_SMD:R_0201_0603Metric
- removed R4, R5: 5k1, Resistor_SMD:R_0603_1608Metric
- added D10: ESD9B5.0ST5G, Diode_SMD:D_SOD-923, F.Cu at (242.0, 70.5)
- added D11: ESD9B5.0ST5G, Diode_SMD:D_SOD-923, F.Cu at (242.0, 72.4)
- added R27: 5k1, Resistor_SMD:R_0603_1608Metric, F.Cu at (242.6, 65.8)
- added R52: 33R, Resistor_SMD:R_0603_1608Metric, F.Cu at (242.6, 68.3)
- added U9: NHD-2.4-240320AF-CSXP, Display:EA_eDIPTFT32-XXX, F.Cu at (185.4, 78.8)
- R40: value 33R -> 5k1
Connections:
- R40 pad 1: Net-(U1-IO15) -> GND
- R40 pad 2: /SD_CS -> Net-(J6-CC1)
- U1 pad 10: /ATM_IRQ -> unconnected-(U1-IO25-Pad10)
- U1 pad 11: /ATM_WO -> /SD_MISO
- U1 pad 12: /ATM_ZX -> Net-(U1-IO27)
- U1 pad 14: /SD_MISO -> unconnected-(U1-IO12-Pad14)
- U1 pad 23: Net-(U1-IO15) -> unconnected-(U1-IO15-Pad23)
- U1 pad 24: /DSP_BRIGHT -> unconnected-(U1-IO2-Pad24)
- U1 pad 6: unconnected-(U1-IO34-Pad6) -> /ATM_CF1
- U1 pad 7: unconnected-(U1-IO35-Pad7) -> /ATM_IRQ
- U1 pad 8: /ATM_CF2 -> /ATM_ZX
- U1 pad 9: /ATIM_CF1 -> /DSP_BRIGHT
- U4 pad 17: /ATM_WO -> unconnected-(U4-WarnOut-Pad17)
- U4 pad 19: /ATM_CF2 -> unconnected-(U4-CF2-Pad19)

Commit message: Uradjeno pola rutiranja
Parts:
- removed D5: BAT760, Diode_SMD:D_SOD-323
- removed D9: LED_ORANGE, LED_SMD:LED_0805_2012Metric
- removed R10: 330R, Resistor_SMD:R_0603_1608Metric
- removed R12: 56k, Resistor_SMD:R_0603_1608Metric
- removed R14, R23: 20R, Resistor_SMD:R_0805_2012Metric
- removed R15, R6: 10R, Resistor_SMD:R_0805_2012Metric
- removed R42: 22k1, Resistor_SMD:R_0603_1608Metric
- removed R64: 10k, Resistor_SMD:R_0603_1608Metric
- removed U9: NHD-2.4-240320AF-CSXP, Display:EA_eDIPTFT32-XXX
- added J6: USB4110-GF-A, USB4110-GF-A-foot:USB4110-GF-A_GCT, F.Cu at (34.8, 115.0)
- added TP4: TestPoint, test_points:TestPoint_Pad_D2.0mm, F.Cu at (122.5, 119.5)
- C37: footprint Capacitor_SMD:CP_Elec_16x22 -> Capacitor_SMD:CP_Elec_16x17.5
- J2: footprint 2073-MEM2067-02-180-00-ACT-ND:CONN_MEM2067-02-180-00-A_GCT -> usb:CONN_MEM2067-02-180-00-A_GCT
- JP1, JP2: footprint Jumper:SolderJumper-3_P1.3mm_Bridged12_Pad1.0x1.5mm -> Jumper:SolderJumper-3_P1.3mm_Bridged12_RoundedPad1.0x1.5mm
- SW2: footprint blue:SWITCH_43SMTR92LFS -> red:SWITCH_45SK43SMTR92LFS
- SW3: footprint CKN9112CT-ND_sw:SWITCH_43SMTR92LFS -> blue:SWITCH_43SMTR92LFS
- TP1, TP2, TP3, TP6: footprint TestPoint:TestPoint_Pad_D2.0mm -> test_points:TestPoint_Pad_D2.0mm
- U1: footprint RF_Module:ESP32-WROOM-32D -> esp32_custom:ESP32-WROOM-32D
- moved R27 206.4 mm to (42.2, 115.1)
- moved D10 205.0 mm to (41.6, 113.6)
- moved D11 203.3 mm to (42.6, 112.0)
- moved R52 139.6 mm to (103.0, 68.3), turned to 90 degrees
- moved Q3 36.0 mm to (116.6, 133.1), turned to 180 degrees
- moved R54 32.0 mm to (106.5, 102.8), turned to 90 degrees
- moved R53 31.4 mm to (112.5, 118.8), turned to -90 degrees
- moved R62 29.7 mm to (121.0, 133.0), turned to 90 degrees
- moved R63 27.6 mm to (109.5, 120.8)
- moved D2 27.1 mm to (40.6, 122.6)
- moved C49 25.7 mm to (74.7, 125.0)
- moved R33 24.9 mm to (72.2, 122.1), turned to 180 degrees
- moved C48 24.1 mm to (117.2, 120.0)
- moved R35 23.2 mm to (65.5, 104.5), turned to 180 degrees
- moved R57 22.3 mm to (110.2, 107.5), turned to 180 degrees
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Connections:
- C11 pad 1: +3.3VA -> +3.3VD
- C16 pad 2: GND -> GNDA
- C18 pad 2: GND -> GNDA
- C19 pad 1: GND -> GNDA
- C26 pad 2: GND -> GNDA
- C36 pad 2: GND -> GNDA
- C38 pad 2: +3.3VA -> +3.3VD
- C41 pad 2: GND -> GNDA
- C44 pad 1: GND -> GNDA
- C44 pad 2: Net-(U4-AVDD) -> +3.3VA
- R17 pad 2: GND -> GNDA
- R18 pad 1: GND -> GNDA
- R24 pad 1: GND -> GNDA
- R34 pad 1: GND -> GNDA
- R35 pad 1: Net-(U4-AVDD) -> GND
- R35 pad 2: +3.3VA -> GNDA
- U4 pad 14: GND -> GNDA
- U4 pad 3: +3.3VA -> +3.3VD
- U4 pad 5: Net-(U4-AVDD) -> +3.3VA
- U4 pad 6: GND -> GNDA
- U4 pad 7: GND -> GNDA
- U4 pad 8: GND -> GNDA
Routing:
- net +3.3VD: track 0.00 -> 392.9 mm
- net +5V: track 0.00 -> 98.8 mm
- net V_IN: track 0.00 -> 62.9 mm
- net /SD_MOSI: track 0.00 -> 53.9 mm
- net Net-(U1-IO14): track 0.00 -> 46.7 mm
- net +7V rectified: track 0.00 -> 41.6 mm
- net /RTS: track 0.00 -> 39.0 mm
- net Net-(J2-DAT0): track 0.00 -> 38.0 mm
- net /SD_CS: track 0.00 -> 35.3 mm
- net /SD_SCLK: track 0.00 -> 33.4 mm
- net +3.3VA: track 0.00 -> 32.5 mm
- net /VBUS-3.3: track 0.00 -> 30.1 mm
- net /LED-K1: track 0.00 -> 27.6 mm
- net /DTR: track 0.00 -> 24.8 mm
- net N: track 0.00 -> 22.3 mm
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- added copper zone on B.Cu, net GND
- added copper zone on B.Cu, net GNDA
Other:
- board text removed: "Footprint se ne poklapa sa simbolom i mora ili footprint ili simbol ručno da se promeni."

Commit message: Uradjen PCB
Parts:
- removed R35: 0R, Resistor_SMD:R_0603_1608Metric
- removed R53: 10k, Resistor_SMD:R_0603_1608Metric
- added R43: 33R, Resistor_SMD:R_0603_1608Metric, F.Cu at (72.0, 104.2)
- added R47: 33R, Resistor_SMD:R_0603_1608Metric, F.Cu at (72.0, 107.8)
- added R65: 33R, Resistor_SMD:R_0603_1608Metric, F.Cu at (72.0, 110.2)
- moved SW3 110.8 mm to (58.0, 20.5), turned to 90 degrees
- moved J6 110.5 mm to (89.5, 19.0), turned to 180 degrees
- moved SW2 106.7 mm to (66.2, 20.5)
- moved D2 101.2 mm to (79.5, 29.2), turned to 90 degrees
- moved R31 100.5 mm to (83.6, 29.4), turned to -90 degrees
- moved C49 99.2 mm to (59.7, 27.0)
- moved D10 99.0 mm to (89.5, 27.0)
- moved C17 98.8 mm to (86.3, 29.7), turned to -90 degrees
- moved D11 98.0 mm to (93.0, 28.0), turned to 180 degrees
- moved R27 97.6 mm to (89.3, 29.7), turned to -90 degrees
- moved R56 97.0 mm to (54.9, 27.5)
- moved R32 95.9 mm to (83.6, 32.9), turned to -90 degrees
- moved SW1 91.5 mm to (74.7, 20.5), turned to 90 degrees
- moved R26 81.8 mm to (89.5, 39.2), turned to 90 degrees
- moved R28 80.8 mm to (91.5, 39.2), turned to 90 degrees
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Connections:
- C16 pad 2: GNDA -> GND
- C18 pad 2: GNDA -> GND
- C19 pad 1: GNDA -> GND
- C26 pad 2: GNDA -> GND
- C36 pad 2: GNDA -> GND
- C41 pad 2: GNDA -> GND
- C44 pad 1: GNDA -> GND
- R17 pad 2: GNDA -> GND
- R18 pad 1: GNDA -> GND
- R24 pad 1: GNDA -> GND
- R34 pad 1: GNDA -> GND
- U1 pad 26: /random -> unconnected-(U1-IO4-Pad26)
- U4 pad 14: GNDA -> GND
- U4 pad 18: /ATIM_CF1 -> Net-(U4-CF1)
- U4 pad 20: /ATM_IRQ -> Net-(U4-IRQ)
- U4 pad 21: /ATM_ZX -> Net-(U4-ZX)
- U4 pad 6: GNDA -> GND
- U4 pad 7: GNDA -> GND
- U4 pad 8: GNDA -> GND
- U6 pad 4: /Data+ -> /D+
- U6 pad 5: /Data- -> /D-
Routing:
- net /IO0: track 13.8 -> 112.2 mm, vias 0 -> 2
- net /ATM_CF1: track 0.00 -> 93.5 mm, vias 0 -> 6
- net /ATM_IRQ: track 0.00 -> 91.4 mm, vias 0 -> 6
- net /ATM_ZX: track 0.00 -> 90.2 mm, vias 0 -> 6
- net VBUS: track 18.9 -> 102.2 mm, vias 0 -> 2
- net /EN: track 8.43 -> 89.6 mm, vias 0 -> 4
- net /SCLK: track 0.00 -> 81.1 mm, vias 0 -> 2
- net /MOSI: track 0.00 -> 80.9 mm, vias 0 -> 2
- net /RXD0: track 0.00 -> 64.8 mm, vias 0 -> 2
- net /TXD0: track 0.00 -> 61.9 mm, vias 0 -> 2
- net /MISO: track 3.75 -> 57.5 mm, vias 0 -> 2
- net +3.3VD: track 392.9 -> 344.7 mm, vias 0 -> 6
- net GND: track 0.00 -> 47.7 mm, vias 0 -> 43
- net /ATM_CS: track 0.00 -> 47.1 mm
- net /DSP_RESX: track 0.00 -> 45.1 mm, vias 0 -> 2
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- added copper zone on F.Cu, net GND
- removed copper zone on B.Cu, net GNDA
Other:
- board size 150 x 150 mm -> 102 x 103 mm

Commit message: Generisani Gerber i Drill
Parts:
- removed J2: MEM2067-02-180-00-A, usb:CONN_MEM2067-02-180-00-A_GCT
- added J1: MEM2067-02-180-00-A_REVB, MEM2067-02-180-00-A_REVB_foot:GCT_MEM2067-02-180-00-A_REVB, F.Cu at (106.0, 21.5)
- J3: footprint PJ_002AH:PJ-002AH-SMT-TR_CUD -> CUI_PJ-002AH-SMT-TR-foot:CUI_PJ-002AH-SMT-TR
- J4: footprint SJ_3523_SMT:SJ-3523-SMT_CUD -> CUI_SJ-3523-SMT-TR-foot:CUI_SJ-3523-SMT-TR
- J5: footprint 541324062:CON_541324062_MOL -> Molex0541324062-foot:CON_541324062_MOL
- U1: footprint esp32_custom:ESP32-WROOM-32D -> RF_Module:ESP32-WROOM-32D
- U8: footprint TPS2121RUXR:RUX0012A -> TPS2121RUXR-foot:RUX0012A
- moved J3 8.77 mm to (30.3, 76.3), turned to 90 degrees
- moved J4 0.73 mm to (36.3, 99.9), turned to 90 degrees
Routing:
- net N: track 30.4 -> 40.6 mm
- net L: track 26.5 -> 33.1 mm
- net Net-(J4-TIP): track 4.90 -> 5.68 mm
- net /ATM_CF1: vias 6 -> 2
- net /ATM_ZX: vias 6 -> 2
- net /ATM_IRQ: vias 6 -> 2
- net GND: vias 43 -> 102
- net (no net): vias 79 -> 1
Other:
- board text added: "Designed by 4 DIGITALCA"
